File: PCB/kicad/USB-HUB(SL2.1A).kicad_sch (KiCad schematic)
At the start: 33 parts, among them U1 SL2.1S

Commit message: rev 2.0
Parts:
- removed C9: 100nF, Capacitor_SMD:C_0402_1005Metric, symbol Device:C
- added C15, C17: 10uF, Capacitor_SMD:C_0402_1005Metric, symbol Device:C
- added C16, C18: 100nF, Capacitor_SMD:C_0402_1005Metric, symbol Device:C
- added C19, C20: 1uF, Capacitor_SMD:C_0402_1005Metric, symbol Device:C
- added D2, D3, D4, D5, D6: LED, LED_SMD:LED_0402_1005Metric, symbol Device:LED
- added H1, H2, H3, H4: MountingHole_Pad_MP, MountingHole:MountingHole_2.5mm_Pad_TopBottom, symbol Mechanical:MountingHole_Pad_MP
- added J1, J2, J3, J4: USB_A, easyeda2kicad:USB-A-TH_10.0QHHTZB6.3, symbol Connector:USB_A
- added R13, R14, R15, R16: 5.1K, Resistor_SMD:R_0402_1005Metric, symbol Device:R
- added SW1: SW_Push_45deg, Resistor_SMD:R_0402_1005Metric, symbol Switch:SW_Push_45deg
- added U2: SL2.1S, easyeda2kicad:SSOP-16_L4.6-W2.6-P0.53-LS4.0-BL, symbol easyeda2kicad:SL2.1S
- added U3: MCP2221AxML, Package_DFN_QFN:QFN-16-1EP_4x4mm_P0.65mm_EP2.5x2.5mm, symbol Interface_USB:MCP2221AxML
- C10, C11, C12, C13, C14: LCSC Part C28323 -> C14445
- C5, C6, C7, C8: value 100nF -> 1uF; LCSC Part C1525 -> C14445
Connections:
- net D1+: now also J3.3 (D+); no longer USB2.6 (DP1), USB2.8 (DP2)
- net D1-: now also J3.2 (D-); no longer USB2.5 (DN2), USB2.7 (DN1)
- net D2+: now also USB2.6 (DP1), USB2.8 (DP2); no longer USB3.6 (DP1), USB3.8 (DP2)
- net D2-: now also USB2.5 (DN2), USB2.7 (DN1); no longer USB3.5 (DN2), USB3.7 (DN1)
- net D3+: now also U2.6 (UDP); no longer USB4.6 (DP1), USB4.8 (DP2)
- net D3-: now also U2.5 (UDM); no longer USB4.5 (DN2), USB4.7 (DN1)
- net D4+: now also J4.3 (D+); no longer USB5.6 (DP1), USB5.8 (DP2)
- net D4-: now also J4.2 (D-); no longer USB5.5 (DN2), USB5.7 (DN1)
- net GND: now also C15.2, C16.2, C17.2, C18.2, C19.2, C20.2, D6.1 (K), H1.MP, H2.MP, H3.MP, H4.MP, J1.4 (GND), J1.5 (Shield), J2.4 (GND), J2.5 (Shield), J3.4 (GND), J3.5 (Shield), J4.4 (GND), J4.5 (Shield), SW1.2, U2.12 (XIN), U2.8 (VSS), U3.13 (VSS)
- net VBUS: now also C20.1, D2.2 (A), D3.2 (A), D4.2 (A), D5.2 (A), J1.1 (VBUS), J2.1 (VBUS), J3.1 (VBUS), J4.1 (VBUS), U2.7 (VDD5), U3.16 (VDD)
- new net: C17.1, C18.1, U2.10 (VDD18)
- new net: D4.1 (K), R15.2
- new net: D5.1 (K), D6.2 (A), R16.2
- new net: D3.1 (K), R14.2
- new net: SW1.1, U3.3 (~{RST})
- new net: C19.1, U3.10 (VUSB)
- new net: D2.1 (K), R13.2
- new net: C15.1, C16.1, U2.9 (VDD33)
- new net D5+: U2.4 (DP1), USB5.6 (DP1), USB5.8 (DP2)
- new net D5-: U2.3 (DM1), USB5.5 (DN2), USB5.7 (DN1)
- new net D6+: U2.2 (DP2), USB4.6 (DP1), USB4.8 (DP2)
- new net D6-: U2.1 (DM2), USB4.5 (DN2), USB4.7 (DN1)
- new net D7+: U2.16 (DP3), USB3.6 (DP1), USB3.8 (DP2)
- new net D7-: U2.15 (DM3), USB3.5 (DN2), USB3.7 (DN1)
- new net D8+: U2.14 (DP4), U3.12 (D+)
- new net D8-: U2.13 (DM4), U3.11 (D-)
- new net LED_I2C: R15.1, U3.7 (GP3)
- new net LED_URX: R13.1, U3.1 (GP0)
- new net LED_UTX: R14.1, U3.2 (GP1)
- new net SCL: J2.3 (D+), U3.9 (SCL)
- new net SDA: J2.2 (D-), U3.8 (SDA)
- new net URX: J1.3 (D+), U3.4 (URx)
- new net USB_CFG: R16.1, U3.6 (GP2)
- new net UTX: J1.2 (D-), U3.5 (UTx)
- no-connect marks 11 -> 12
Other:
- moved on the sheet: C1, C11, C12, C13, C14, C2, C3, C4, R10, R3, R4, R5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
